File: Hardware/SparkFun_Analog_MEMS_Microphone_Breakout_ICS40180.brd (EAGLE design)
At the start: 14 x 10.2 mm, 25 parts, among them U1 OPA344, U2 ICS40180

Commit message: Migrating mic and VCC/GNDs to latest eagle libraries
-Doesn't change design at all, but just makes it cleaner/easier to know where the devices live in our main eagle libraries repo.
Parts:
- U2: device ICS-40180:ICS40180 -> SparkFun-Sensors:ICS40180
Changed lines of the file:
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@@
 <drawing>
 <settings>
-<setting alwaysvectorfont="yes"/>
+<setting alwaysvectorfont="no"/>
 <setting keepoldvectorfont="yes"/>
 <setting verticaltext="up"/>
@@
 <layer number="47" name="Measures" color="7" fill="1" visible="no" active="yes"/>
 <layer number="48" name="Document" color="7" fill="1" visible="no" active="yes"/>
-<layer number="49" name="Reference" color="7" fill="1" visible="yes" active="yes"/>
+<layer number="49" name="Reference" color="7" fill="1" visible="no" active="yes"/>
 <layer number="50" name="dxf" color="7" fill="1" visible="no" active="yes"/>
 <layer number="51" name="tDocu" color="6" fill="1" visible="yes" active="yes"/>
@@
 <attribute name="VALUE" value="1.0uF" x="9.652" y="8.1915" size="0.4064" layer="27" font="vector" ratio="12" rot="R90"/>
 </element>
-<element name="U2" library="ICS-40180" package="ICS40180" value="ICS40180" x="2.54" y="3.81" smashed="yes" rot="R270">
+<element name="U2" library="SparkFun-Sensors" package="ICS40180" value="ICS40180" x="2.54" y="3.81" smashed="yes" rot="R270">
 <attribute name="NAME" x="4.323" y="4.67" size="0.6096" layer="25" font="vector" ratio="20" rot="R270" align="bottom-center"/>
 <attribute name="PROD_ID" value="IC-15819" x="2.54" y="3.81" size="1.778" layer="27" font="vector" ratio="15" rot="R270" display="off"/>
