File: Hardware/SparkFun_Analog_MEMS_Microphone_Breakout_ICS40180.sch (EAGLE design)
At the start: 18 parts, among them U1 OPA344, U2 ICS40180

Commit message: Migrating mic and VCC/GNDs to latest eagle libraries
-Doesn't change design at all, but just makes it cleaner/easier to know where the devices live in our main eagle libraries repo.
Parts:
- U2: device ICS-40180:ICS40180 -> SparkFun-Sensors:ICS40180
Changed lines of the file:
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@@
 <parts>
 <part name="JP1" library="SparkFun-Connectors" deviceset="CONN_03" device="1X03_NO_SILK"/>
-<part name="GND1" library="SparkFun" deviceset="GND" device=""/>
-<part name="P+1" library="SparkFun" deviceset="VCC" device=""/>
-<part name="P+2" library="SparkFun" deviceset="VCC" device=""/>
-<part name="GND2" library="SparkFun" deviceset="GND" device=""/>
-<part name="P+3" library="SparkFun" deviceset="VCC" device=""/>
+<part name="GND1" library="SparkFun-PowerSymbols" deviceset="GND" device=""/>
+<part name="P+1" library="SparkFun-PowerSymbols" deviceset="VCC" device=""/>
+<part name="P+2" library="SparkFun-PowerSymbols" deviceset="VCC" device=""/>
+<part name="GND2" library="SparkFun-PowerSymbols" deviceset="GND" device=""/>
+<part name="P+3" library="SparkFun-PowerSymbols" deviceset="VCC" device=""/>
 <part name="R1" library="SparkFun-Resistors" deviceset="10KOHM" device="-0603-1/10W-1%" value="10k"/>
 <part name="R2" library="SparkFun-Resistors" deviceset="10KOHM" device="-0603-1/10W-1%" value="10k"/>
@@
 <part name="C3" library="SparkFun-Capacitors" deviceset="27PF" device="-0603-50V-5%" value="27pF"/>
 <part name="C4" library="SparkFun-Capacitors" deviceset="0.1UF" device="-0603-25V-(+80/-20%)" value="0.1uF"/>
-<part name="GND3" library="SparkFun" deviceset="GND" device=""/>
-<part name="GND4" library="SparkFun" deviceset="GND" device=""/>
-<part name="P+4" library="SparkFun" deviceset="VCC" device=""/>
-<part name="P+5" library="SparkFun" deviceset="VCC" device=""/>
-<part name="GND5" library="SparkFun" deviceset="GND" device=""/>
+<part name="GND3" library="SparkFun-PowerSymbols" deviceset="GND" device=""/>
+<part name="GND4" library="SparkFun-PowerSymbols" deviceset="GND" device=""/>
+<part name="P+4" library="SparkFun-PowerSymbols" deviceset="VCC" device=""/>
+<part name="P+5" library="SparkFun-PowerSymbols" deviceset="VCC" device=""/>
+<part name="GND5" library="SparkFun-PowerSymbols" deviceset="GND" device=""/>
 <part name="C1" library="SparkFun-Capacitors" deviceset="4.7UF" device="-0603-6.3V-(10%)" value="4.7uF"/>
 <part name="C2" library="SparkFun-Capacitors" deviceset="1.0UF" device="-0603-16V-10%" value="1.0uF"/>
-<part name="U2" library="ICS-40180" deviceset="ICS40180" device=""/>
+<part name="U2" library="SparkFun-Sensors" deviceset="ICS40180" device=""/>
 <part name="U1" library="SparkFun-IC-Amplifiers" deviceset="OPA344" device="" value="OPA344"/>
 <part name="LOGO1" library="SparkFun-Aesthetics" deviceset="SFE_LOGO_FLAME" device=".1_INCH"/>
@@
 <attribute name="VALUE" x="180.34" y="76.2" size="1.778" layer="96" font="vector"/>
 </instance>
-<instance part="P+1" gate="1" x="182.88" y="101.6" smashed="yes">
+<instance part="P+1" gate="G$1" x="182.88" y="101.6" smashed="yes">
 <attribute name="VALUE" x="181.864" y="105.156" size="1.778" layer="96" font="vector"/>
 </instance>
-<instance part="P+2" gate="1" x="195.58" y="127" smashed="yes">
+<instance part="P+2" gate="G$1" x="195.58" y="127" smashed="yes">
 <attribute name="VALUE" x="194.564" y="130.556" size="1.778" layer="96" font="vector"/>
 </instance>
@@
 <attribute name="VALUE" x="193.04" y="111.76" size="1.778" layer="96" font="vector"/>
 </instance>
-<instance part="P+3" gate="1" x="50.8" y="127" smashed="yes">
+<instance part="P+3" gate="G$1" x="50.8" y="127" smashed="yes">
 <attribute name="VALUE" x="49.784" y="130.556" size="1.778" layer="96" font="vector"/>
 </instance>
@@
 <attribute name="VALUE" x="154.94" y="73.66" size="1.778" layer="96" font="vector"/>
 </instance>
-<instance part="P+4" gate="1" x="160.02" y="111.76" smashed="yes">
+<instance part="P+4" gate="G$1" x="160.02" y="111.76" smashed="yes">
 <attribute name="VALUE" x="159.004" y="115.316" size="1.778" layer="96" font="vector"/>
 </instance>
-<instance part="P+5" gate="1" x="35.56" y="127" smashed="yes">
+<instance part="P+5" gate="G$1" x="35.56" y="127" smashed="yes">
 <attribute name="VALUE" x="34.544" y="130.556" size="1.778" layer="96" font="vector"/>
 </instance>
@@
 <wire x1="195.58" y1="124.46" x2="195.58" y2="127" width="0.1524" layer="91"/>
 <pinref part="JP1" gate="J$1" pin="1"/>
-<pinref part="P+2" gate="1" pin="VCC"/>
+<pinref part="P+2" gate="G$1" pin="VCC"/>
 </segment>
 <segment>
 <wire x1="50.8" y1="127" x2="50.8" y2="124.46" width="0.1524" layer="91"/>
 <wire x1="53.34" y1="124.46" x2="50.8" y2="124.46" width="0.1524" layer="91"/>
-<pinref part="P+3" gate="1" pin="VCC"/>
+<pinref part="P+3" gate="G$1" pin="VCC"/>
 <pinref part="U2" gate="G$1" pin="VDD"/>
 </segment>
@@
 <wire x1="160.02" y1="109.22" x2="160.02" y2="111.76" width="0.1524" layer="91"/>
 <pinref part="R1" gate="G$1" pin="2"/>
-<pinref part="P+4" gate="1" pin="VCC"/>
+<pinref part="P+4" gate="G$1" pin="VCC"/>
 </segment>
 <segment>
 <wire x1="182.88" y1="99.06" x2="182.88" y2="101.6" width="0.1524" layer="91"/>
-<pinref part="P+1" gate="1" pin="VCC"/>
+<pinref part="P+1" gate="G$1" pin="VCC"/>
 <pinref part="U1" gate="G2" pin="P$V+"/>
 </segment>
@@
 <wire x1="35.56" y1="124.46" x2="35.56" y2="127" width="0.1524" layer="91"/>
 <pinref part="C4" gate="G$1" pin="2"/>
-<pinref part="P+5" gate="1" pin="VCC"/>
+<pinref part="P+5" gate="G$1" pin="VCC"/>
 </segment>
 </net>
